File: KiCad_pour_PCB/PCB_Plaque_Basse/PCB_Plaque_Basse.kicad_sch (KiCad schematic)
At the start: 9 parts

Commit message: Avancement carte PCB
Parts:
- removed BMP1: ~, INSARIANNE_Lib:BMP180, symbol INSARIANNE_Lib:BMP180
- removed Bloc_pile1: ~, Connector_PinHeader_1.00mm:PinHeader_1x02_P1.00mm_Vertical, symbol INSARIANNE_Lib:Bloc_pile
- removed Inter_Input1: ~, Connector_PinHeader_1.00mm:PinHeader_1x06_P1.00mm_Vertical, symbol INSARIANNE_Lib:Interface_input
- removed MPU1: ~, INSARIANNE_Lib:MPU6050, symbol INSARIANNE_Lib:MPU6050
- removed Servomoteur1, Servomoteur2: ~, Connector_PinHeader_1.00mm:PinHeader_1x03_P1.00mm_Vertical, symbol INSARIANNE_Lib:Servomoteur
- added Module_LORA1: ~, symbol INSARIANNE_Lib:Module_LORA
- added Module_SD1: ~, symbol INSARIANNE_Lib:Module_SD
Connections:
- net at Inter_plaques1.1 (5V): now also Arduino_Nano1.27 (5V), Module_LORA1. (VDD), Module_SD1. (SCK)
- net at Arduino_Nano1.29 (GND), Inter_plaques1.2 (GND): now also Module_LORA1. (VDD), Module_SD1. (SCK)
- net at Inter_plaques1.4 (A5): now also Arduino_Nano1.24 (A5)
- net at Inter_plaques1.5 (A4): now also Arduino_Nano1.23 (A4)
- net at Arduino_Nano1.14 (D11): now also Module_LORA1. (VDD), Module_SD1. (SCK)
- net at Arduino_Nano1.15 (D12): now also Module_LORA1. (VDD), Module_SD1. (SCK)
- net at Arduino_Nano1.16 (D13): now also Module_LORA1. (VDD), Module_SD1. (SCK)
- net at Arduino_Nano1.8 (D5): now also Module_LORA1. (VDD)
- net at Arduino_Nano1.9 (D6): now also Module_SD1. (SCK)
- no-connect marks 24 -> 29
Other:
- company: INS'AERO - PÔLE TECHNIQUE - INSA CVL -> (none)
- title: INSARIANNE1 Haute - v3 -> (none)

Commit message: PCB_Fin
Parts:
- Module_LORA1: footprint (none) -> INSARIANNE_Lib:Module_LORA
- Module_SD1: footprint (none) -> INSARIANNE_Lib:Module_SD
Connections:
- net at Arduino_Nano1.27 (5V), Inter_plaques1.1 (5V): now also Module_LORA1.4 (VDD), Module_SD1.3 (5V); no longer Module_LORA1. (VDD), Module_SD1. (SCK)
- net at Arduino_Nano1.29 (GND), Inter_plaques1.2 (GND): now also Module_LORA1.7 (GND), Module_SD1.1 (GND); no longer Module_LORA1. (VDD), Module_SD1. (SCK)
- net at Arduino_Nano1.9 (D6): now also Module_SD1.4 (CS); no longer Module_SD1. (SCK)
- net at Arduino_Nano1.8 (D5): now also Module_LORA1.13 (NSS); no longer Module_LORA1. (VDD)
- new net: Arduino_Nano1.14 (D11), Module_LORA1.11 (MOSI), Module_SD1.5 (MOSI)
- new net: Arduino_Nano1.16 (D13), Module_LORA1.12 (SCK), Module_SD1.6 (SCK)
- new net: Arduino_Nano1.15 (D12), Module_LORA1.10 (MISO), Module_SD1.7 (MISO)
Changed lines of the file:
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@@
+	)
+	(no_connect
+		(at 88.9 74.93)
 	)
 	(no_connect
@@
 	)
 	(no_connect
-		(at 99.06 72.39)
-	)
-	(no_connect
 		(at 99.06 67.31)
 	)
@@
 	(wire
 		(pts
-			(xy 90.17 74.93) (xy 90.17 80.01)
-		)
-		(stroke
-			(width 0)
-			(type default)
-		)
-	)
-	(wire
-		(pts
 			(xy 90.17 63.5) (xy 90.17 62.23)
 		)
@@
 	(wire
 		(pts
+			(xy 97.79 72.39) (xy 99.06 72.39)
+		)
+		(stroke
+			(width 0)
+			(type default)
+		)
+	)
+	(wire
+		(pts
 			(xy 125.73 144.78) (xy 125.73 149.86)
 		)
@@
 	(wire
 		(pts
-			(xy 90.17 80.01) (xy 129.54 80.01)
+			(xy 97.79 80.01) (xy 129.54 80.01)
 		)
 		(stroke
@@
 	(wire
 		(pts
-			(xy 88.9 74.93) (xy 90.17 74.93)
-		)
-		(stroke
-			(width 0)
-			(type default)
-		)
-	)
-	(wire
-		(pts
 			(xy 158.75 127) (xy 185.42 127)
+		)
+		(stroke
+			(width 0)
+			(type default)
+		)
+	)
+	(wire
+		(pts
+			(xy 97.79 72.39) (xy 97.79 80.01)
 		)
 		(stroke
@@
 			)
 		)
-		(property "Footprint" ""
+		(property "Footprint" "INSARIANNE_Lib:Module_SD"
 			(at 138.43 53.34 0)
 			(effects
@@
 			)
 		)
-		(pin ""
-		)
-		(pin ""
-		)
-		(pin ""
-		)
-		(pin ""
-		)
-		(pin ""
-		)
-		(pin ""
-		)
-		(pin ""
-		)
-		(pin ""
+		(pin "2"
+		)
+		(pin "3"
+		)
+		(pin "8"
+		)
+		(pin "7"
+		)
+		(pin "1"
+		)
+		(pin "6"
+		)
+		(pin "5"
+		)
+		(pin "4"
 		)
 		(instances
@@
 			)
 		)
-		(property "Footprint" ""
+		(property "Footprint" "INSARIANNE_Lib:Module_LORA"
 			(at 93.98 80.01 0)
 			(effects
@@
 			)
 		)
-		(pin ""
-		)
-		(pin ""
-		)
-		(pin ""
-		)
-		(pin ""
-		)
-		(pin ""
-		)
-		(pin ""
-		)
-		(pin ""
-		)
-		(pin ""
-		)
-		(pin ""
-		)
-		(pin ""
-		)
-		(pin ""
-		)
-		(pin ""
-		)
-		(pin ""
-		)
-		(pin ""
-		)
-		(pin ""
-		)
-		(pin ""
+		(pin "8"
+		)
+		(pin "3"
+		)
+		(pin "11"
+		)
+		(pin "6"
+		)
+		(pin "12"
+		)
+		(pin "7"
+		)
+		(pin "13"
+		)
+		(pin "10"
+		)
+		(pin "2"
+		)
+		(pin "14"
+		)
+		(pin "4"
+		)
+		(pin "5"
+		)
+		(pin "16"
+		)
+		(pin "15"
+		)
+		(pin "1"
+		)
+		(pin "9"
 		)
 		(instances

Commit message: Nouvelle version PCB _ Suite RCE3
Parts:
- removed Inter_in_c1: ~, Connector_PinHeader_1.00mm:PinHeader_1x03_P1.00mm_Vertical, symbol INSARIANNE_Lib:Interface_in_c2
- removed Inter_plaques1: ~, Connector_PinHeader_1.00mm:PinHeader_1x05_P1.00mm_Vertical, symbol INSARIANNE_Lib:Interface_Phaute_Pbasse
- removed Module_SD1: ~, INSARIANNE_Lib:Module_SD, symbol INSARIANNE_Lib:Module_SD
- added BMP1: ~, INSARIANNE_Lib:BMP180, symbol INSARIANNE_Lib:BMP180
- added Inter_Cap_Vol1: ~, Connector_PinHeader_2.54mm:PinHeader_1x02_P2.54mm_Vertical, symbol INSARIANNE_Lib:Interface_Cap_Vol
- added Inter_Pile1: ~, Connector_PinHeader_2.54mm:PinHeader_1x02_P2.54mm_Vertical, symbol INSARIANNE_Lib:Inter_pile
- added MPU1: ~, INSARIANNE_Lib:MPU6050, symbol INSARIANNE_Lib:MPU6050
Connections:
- net at Arduino_Nano1.29 (GND), Module_LORA1.7 (GND): now also BMP1.2 (GND), Inter_Pile1.1 (GND), MPU1.2 (GND)
- net at Arduino_Nano1.27 (5V), Module_LORA1.4 (VDD): now also BMP1.1 (VCC), Inter_Cap_Vol1.1 (GND), MPU1.1 (VCC)
- net at Arduino_Nano1.30 (Vin): now also Inter_Pile1.2 (Vin)
- net at Arduino_Nano1.24 (A5): now also BMP1.3 (SCL), MPU1.3 (SCL)
- net at Arduino_Nano1.23 (A4): now also BMP1.4 (SDA), MPU1.4 (SDA)
- net at Arduino_Nano1.7 (D4): now also Inter_Cap_Vol1.2 (Cap)
- no-connect marks 29 -> 34
