File: KiCad_pour_PCB/PCB_Plaque_Basse/PCB_Plaque_Basse.kicad_pcb (KiCad board)
At the start: 2 copper layers, 108 x 108 mm, 3 parts

Commit message: PCB_Fin
Parts:
- added Module_LORA1: ~, INSARIANNE_Lib:Module_LORA, F.Cu at (171.3, 99.8)
- added Module_SD1: ~, INSARIANNE_Lib:Module_SD, F.Cu at (152.8, 141.8)
- moved Inter_in_c1 73.5 mm to (158.3, 60.2), turned to 0 degrees
- moved Inter_plaques1 33.4 mm to (162.8, 66.8), turned to -90 degrees
- moved Arduino_Nano1 22.3 mm to (148.9, 64.6), turned to 180 degrees
Routing:
- net Net-(Arduino_Nano1-D11): track 0.00 -> 148.6 mm
- net Net-(Arduino_Nano1-D12): track 0.00 -> 111.5 mm
- net Net-(Arduino_Nano1-D13): track 0.00 -> 93.3 mm
- net Net-(Arduino_Nano1-D5): track 0.00 -> 85.1 mm
- net Net-(Arduino_Nano1-5V): track 0.00 -> 64.7 mm
- net Net-(Inter_plaques1-GND): track 0.00 -> 50.7 mm
- net Net-(Arduino_Nano1-D6): track 0.00 -> 34.8 mm
- net Net-(Arduino_Nano1-A4): track 0.00 -> 34.3 mm
- net Net-(Arduino_Nano1-A5): track 0.00 -> 33.9 mm
- net Net-(Arduino_Nano1-D4): track 0.00 -> 26.5 mm
- net Net-(Arduino_Nano1-D3): track 0.00 -> 23.6 mm
- net Net-(Arduino_Nano1-D2): track 0.00 -> 20.6 mm
- net Net-(Arduino_Nano1-Vin): track 0.00 -> 18.1 mm
- added copper zone on B.Cu, net Net-(Inter_plaques1-GND)
- added copper zone on F.Cu, net Net-(Inter_plaques1-GND)
Other:
- board size 108 x 108 mm -> 94 x 94 mm

Commit message: Nouvelle version PCB _ Suite RCE3
Parts:
- removed Inter_in_c1: ~, Connector_PinHeader_1.00mm:PinHeader_1x03_P1.00mm_Vertical
- removed Inter_plaques1: ~, Connector_PinHeader_1.00mm:PinHeader_1x05_P1.00mm_Vertical
- added BMP1: ~, INSARIANNE_Lib:BMP180, F.Cu at (119.8, 109.3)
- added Inter_Cap_Vol1: ~, Connector_PinHeader_2.54mm:PinHeader_1x02_P2.54mm_Vertical, F.Cu at (160.5, 68.3)
- added Inter_Pile1: ~, Connector_PinHeader_2.54mm:PinHeader_1x02_P2.54mm_Vertical, F.Cu at (160.5, 75.7)
- added MPU1: ~, INSARIANNE_Lib:MPU6050, F.Cu at (116.3, 90.3)
- moved Module_LORA1 5.45 mm to (174.0, 95.0)
Connections:
- Arduino_Nano1 pad 4: unconnected-(Arduino_Nano1-GND-Pad4) -> Net-(Inter_Cap_Vol1-GND)
- Arduino_Nano1 pad 5: Net-(Arduino_Nano1-D2) -> unconnected-(Arduino_Nano1-D2-Pad5)
- Arduino_Nano1 pad 6: Net-(Arduino_Nano1-D3) -> unconnected-(Arduino_Nano1-D3-Pad6)
Routing:
- net Net-(BMP1-GND): track 50.7 -> 101.9 mm
- net Net-(Arduino_Nano1-5V): track 64.7 -> 89.0 mm
- net Net-(Arduino_Nano1-D3): track 23.6 -> 0.00 mm
- net Net-(Inter_Cap_Vol1-GND): track 0.00 -> 21.7 mm
- net Net-(Arduino_Nano1-D2): track 20.6 -> 0.00 mm
- net Net-(Arduino_Nano1-A5): track 33.9 -> 49.3 mm
- net Net-(Arduino_Nano1-A4): track 34.3 -> 49.0 mm
- net Net-(Arduino_Nano1-Vin): track 18.1 -> 12.3 mm
- net Net-(Arduino_Nano1-D11): track 148.6 -> 143.9 mm
- net Net-(Arduino_Nano1-D5): track 85.1 -> 80.8 mm
- net Net-(Arduino_Nano1-D4): track 26.5 -> 30.5 mm
- net Net-(Arduino_Nano1-D13): track 93.3 -> 90.7 mm
- net Net-(Arduino_Nano1-D12): track 111.5 -> 109.6 mm

Commit message: Fin carte PCB
Other:
- board text added: "2023/2024"
- board text added: "INS'aéro"
- board text added: "PCB_Plaque_Basse INSARIANNE1"
Changed lines of the file:
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@@
 		(tags "Through hole pin header THT 1x02 2.54mm single row")
 		(property "Reference" "Inter_Pile1"
-			(at 0 -2.725 360)
+			(at 0 -2.725 0)
 			(layer "F.SilkS")
 			(effects
@@
 		)
 		(property "Value" "~"
-			(at 0 4.87 360)
+			(at 0 4.87 0)
 			(layer "F.Fab")
 			(hide yes)
@@
 		(layer "User.2")
 	)
+	(gr_text "2023/2024\n"
+		(at 168 88 0)
+		(layer "F.SilkS")
+		(effects
+			(font
+				(size 1 1)
+				(thickness 0.1)
+			)
+			(justify left bottom)
+		)
+	)
+	(gr_text "PCB_Plaque_Basse\nINSARIANNE1"
+		(at 155.5 86.5 0)
+		(layer "F.SilkS")
+		(effects
+			(font
+				(size 1.5 1.5)
+				(thickness 0.2)
+			)
+			(justify left bottom)
+		)
+	)
+	(gr_text "INS'aéro"
+		(at 155.5 88 0)
+		(layer "F.SilkS")
+		(effects
+			(font
+				(size 1 1)
+				(thickness 0.1)
+			)
+			(justify left bottom)
+		)
+	)
 	(segment
 		(start 148.88 79.88)
@@
 		(polygon
 			(pts
-				(xy 83.5 45) (xy 83.5 151) (xy 83.5 151) (xy 195.5 151) (xy 195.5 45)
+				(xy 83.5 45) (xy 83.5 151) (xy 195.5 151) (xy 195.5 45)
 			)
 		)

Commit message: Correction trous de perçage PCB Truc stupide d'un triangle équilatérales Plus besoin de faire des trous manuellement
Other:
- outline, holes or cut-outs redrawn
Changed lines of the file:
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@@
 	)
 	(gr_circle
-		(center 104.57 124.57)
-		(end 101.57 124.57)
+		(center 100.53 118.63)
+		(end 103.53 118.63)
 		(stroke
 			(width 0.1)
@@
 	)
 	(gr_circle
-		(center 171.07 124.57)
-		(end 168.07 124.57)
+		(center 175.03 118.81)
+		(end 178.03 118.81)
 		(stroke
 			(width 0.1)
@@
 		(fill none)
 		(layer "Edge.Cuts")
+	)
+	(gr_line
+		(start 100.53 118.63)
+		(end 137.83 54.25)
+		(stroke
+			(width 0.1)
+			(type default)
+		)
+		(layer "User.2")
+	)
+	(gr_circle
+		(center 137.83 97.25)
+		(end 159.33 97.25)
+		(stroke
+			(width 0.1)
+			(type default)
+		)
+		(fill none)
+		(layer "User.2")
+	)
+	(gr_line
+		(start 137.83 54.25)
+		(end 175.03 118.81)
+		(stroke
+			(width 0.1)
+			(type default)
+		)
+		(layer "User.2")
 	)
 	(gr_circle
@@
 		(layer "User.2")
 	)
+	(gr_line
+		(start 175.03 118.81)
+		(end 100.53 118.63)
+		(stroke
+			(width 0.1)
+			(type default)
+		)
+		(layer "User.2")
+	)
