File: KiCad_pour_PCB/PCB_Plaque_Haute/PCB_Plaque_Haute.kicad_sch (KiCad schematic)
At the start: 9 parts

Commit message: Nouvelle version PCB _ Suite RCE3
Parts:
- removed BMP1: ~, INSARIANNE_Lib:BMP180, symbol INSARIANNE_Lib:BMP180
- removed Inter_in_c1: ~, Connector_PinHeader_1.00mm:PinHeader_1x03_P1.00mm_Vertical, symbol INSARIANNE_Lib:Interface_in_c2
- removed Inter_plaques1: ~, Connector_PinHeader_1.00mm:PinHeader_1x05_P1.00mm_Vertical, symbol INSARIANNE_Lib:Interface_Phaute_Pbasse
- removed MPU1: ~, INSARIANNE_Lib:MPU6050, symbol INSARIANNE_Lib:MPU6050
- added Inter_Cap_Vol1: ~, Connector_PinHeader_2.54mm:PinHeader_1x02_P2.54mm_Vertical, symbol INSARIANNE_Lib:Interface_Cap_Vol
- added Octocoupleur1: ~, INSARIANNE_Lib:Octocoupleur, symbol INSARIANNE_Lib:Octocoupleur
- Bloc_pile1: footprint Connector_PinHeader_1.00mm:PinHeader_1x02_P1.00mm_Vertical -> Connector_PinHeader_2.54mm:PinHeader_1x02_P2.54mm_Vertical
- Inter_Input1: footprint Connector_PinHeader_1.00mm:PinHeader_1x06_P1.00mm_Vertical -> Connector_PinHeader_2.54mm:PinHeader_1x06_P2.54mm_Vertical
- Servomoteur1, Servomoteur2: footprint Connector_PinHeader_1.00mm:PinHeader_1x03_P1.00mm_Vertical -> Connector_PinHeader_2.54mm:PinHeader_1x03_P2.54mm_Vertical
Connections:
- net at Arduino_Nano1.29 (GND), Bloc_pile1.2 (GND), Inter_Input1.1 (GND)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: now also Octocoupleur1.2 (GND_1)
- net at Arduino_Nano1.11 (D8): now also Octocoupleur1.1 (In_1)
- new net: Inter_Cap_Vol1.2 (Cap), Octocoupleur1.3 (Out_2)
- new net: Inter_Cap_Vol1.1 (5V), Octocoupleur1.4 (5V_2)
- no-connect marks 24 -> 19

Commit message: Fin carte PCB
Connections:
- net at Octocoupleur1.3 (NC): no longer Inter_Cap_Vol1.2 (Cap)
- net at Octocoupleur1.4 (Base): no longer Inter_Cap_Vol1.1 (5V)
- new net: Inter_Cap_Vol1.1 (5V), Octocoupleur1.5 (5V_2)
- new net: Inter_Cap_Vol1.2 (Cap), Octocoupleur1.6 (Out_2)
- no-connect marks 19 -> 21
Changed lines of the file:
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@@
+	)
+	(no_connect
+		(at 140.97 67.31)
 	)
 	(no_connect
@@
 	)
 	(no_connect
+		(at 130.81 72.39)
+	)
+	(no_connect
 		(at 74.93 102.87)
 	)
@@
 	(wire
 		(pts
-			(xy 132.08 68.58) (xy 132.08 69.85)
+			(xy 132.08 67.31) (xy 132.08 68.58)
+		)
+		(stroke
+			(width 0)
+			(type default)
+		)
+	)
+	(wire
+		(pts
+			(xy 138.43 72.39) (xy 138.43 76.2)
 		)
 		(stroke
@@
 	(wire
 		(pts
-			(xy 132.08 73.66) (xy 120.65 73.66)
-		)
-		(stroke
-			(width 0)
-			(type default)
-		)
-	)
-	(wire
-		(pts
 			(xy 124.46 33.02) (xy 116.84 33.02)
 		)
@@
 	(wire
 		(pts
-			(xy 120.65 73.66) (xy 120.65 97.79)
+			(xy 120.65 71.12) (xy 120.65 97.79)
 		)
 		(stroke
@@
 	(wire
 		(pts
-			(xy 130.81 71.12) (xy 132.08 71.12)
+			(xy 130.81 69.85) (xy 132.08 69.85)
 		)
 		(stroke
@@
 	(wire
 		(pts
-			(xy 95.25 69.85) (xy 95.25 78.74)
+			(xy 95.25 68.58) (xy 95.25 78.74)
 		)
 		(stroke
@@
 	(wire
 		(pts
-			(xy 130.81 68.58) (xy 132.08 68.58)
+			(xy 130.81 67.31) (xy 132.08 67.31)
 		)
 		(stroke
@@
 	(wire
 		(pts
-			(xy 140.97 68.58) (xy 135.89 68.58)
+			(xy 120.65 71.12) (xy 132.08 71.12)
 		)
 		(stroke
@@
 	(wire
 		(pts
-			(xy 138.43 71.12) (xy 138.43 76.2)
-		)
-		(stroke
-			(width 0)
-			(type default)
-		)
-	)
-	(wire
-		(pts
 			(xy 73.66 90.17) (xy 73.66 88.9)
 		)
@@
 	(wire
 		(pts
-			(xy 135.89 68.58) (xy 135.89 76.2)
-		)
-		(stroke
-			(width 0)
-			(type default)
-		)
-	)
-	(wire
-		(pts
 			(xy 73.66 91.44) (xy 102.87 91.44)
 		)
@@
 	(wire
 		(pts
+			(xy 135.89 69.85) (xy 135.89 76.2)
+		)
+		(stroke
+			(width 0)
+			(type default)
+		)
+	)
+	(wire
+		(pts
 			(xy 118.11 53.34) (xy 123.19 53.34)
 		)
@@
 	(wire
 		(pts
-			(xy 132.08 69.85) (xy 95.25 69.85)
+			(xy 138.43 72.39) (xy 140.97 72.39)
+		)
+		(stroke
+			(width 0)
+			(type default)
+		)
+	)
+	(wire
+		(pts
+			(xy 132.08 68.58) (xy 95.25 68.58)
 		)
 		(stroke
@@
 	(wire
 		(pts
-			(xy 132.08 71.12) (xy 132.08 73.66)
-		)
-		(stroke
-			(width 0)
-			(type default)
-		)
-	)
-	(wire
-		(pts
-			(xy 140.97 71.12) (xy 138.43 71.12)
+			(xy 132.08 69.85) (xy 132.08 71.12)
+		)
+		(stroke
+			(width 0)
+			(type default)
+		)
+	)
+	(wire
+		(pts
+			(xy 135.89 69.85) (xy 140.97 69.85)
 		)
 		(stroke
@@
 	(symbol
 		(lib_id "INSARIANNE_Lib:Octocoupleur")
-		(at 135.89 64.77 180)
+		(at 135.89 63.5 180)
 		(unit 1)
 		(exclude_from_sim no)
@@
 		(dnp no)
 		(property "Reference" "Octocoupleur1"
-			(at 134.112 64.008 0)
+			(at 134.112 62.738 0)
 			(effects
 				(font
@@
 		)
 		(property "Value" "~"
-			(at 135.89 67.31 0)
+			(at 135.89 66.04 0)
 			(effects
 				(font
@@
 		)
 		(property "Footprint" "INSARIANNE_Lib:Octocoupleur"
-			(at 135.89 64.77 0)
+			(at 135.89 63.5 0)
 			(effects
 				(font
@@
 		)
 		(property "Datasheet" ""
-			(at 135.89 64.77 0)
+			(at 135.89 63.5 0)
 			(effects
 				(font
@@
 		)
 		(property "Description" ""
-			(at 135.89 64.77 0)
+			(at 135.89 63.5 0)
 			(effects
 				(font
@@
 		(pin "4"
 		)
+		(pin "5"
+		)
+		(pin "6"
+		)
 		(instances
